Commit message: urdf updated

File: wafflebot_description/urdf/wafflebot.urdf (robot description, URDF)
Before this commit: robot wafflebot, 7 links, 6 joints
Links:
- link base_link: geometry collision box size=0.140 0.140 0.143; visual mesh filename=package://wafflebot_description/meshes/burger_base.stl scale=0.001 0.001 0.001
- link base_scan: geometry collision cylinder length=0.0315 radius=0.055; visual mesh filename=package://wafflebot_description/meshes/lds.stl scale=0.001 0.001 0.001
- link wheel_left_link: geometry collision cylinder length=0.018 radius=0.033; visual mesh filename=package://wafflebot_description/meshes/left_tire.stl scale=0.001 0.001 0.001
- link wheel_right_link: geometry collision cylinder length=0.018 radius=0.033; visual mesh filename=package://wafflebot_description/meshes/right_tire.stl scale=0.001 0.001 0.001
Joints:
- joint scan_joint: origin xyz=-0.032 0 0.172 rpy=0 0 0 -> xyz=-0.0215 0 0.145 rpy=0 0 0
- joint wheel_left_joint: origin xyz=0.0 0.08 0.023 rpy=-1.57 0 0 -> xyz=-0.051 0.11 0.031 rpy=-1.57 0 0
- joint wheel_right_joint: origin xyz=0.0 -0.080 0.023 rpy=-1.57 0 0 -> xyz=-0.051 -0.11 0.031 rpy=-1.57 0 0
